File: centi-pi'd/centi-pi'd.kicad_sch (KiCad schematic)
At the start: 73 parts, among them IC1 W25Q128JVSIQ, IC2 APS6404L-3SQN-SN, J1 BM03B-SRSS-TBLFSN, J2 Conn_01x20_Socket, J3 Conn_01x20_Socket, J4 TF-115YY-BCP9, Q1 AO3400A, SW1 BOOTSEL, SW2 RESET, U1 RP2350A-QFN60, U2 LD1117S33, Y1 ECS-120-20-33-CKM-TR

Commit message: started layout
Parts:
- removed TP8: Vin, symbol Connector:TestPoint
- removed TP9: USB_Pow, symbol Connector:TestPoint
- C1, C10, C11, C12, C13, C14, C15, C16, C17, C18, C19, C2, C20, C21, C22, C23, C24, C25, C3, C4, C5, C6, C7, C8, C9: footprint Capacitor_THT:CP_Radial_D5.0mm_P2.00mm -> Capacitor_SMD:C_0603_1608Metric
- D1: footprint (none) -> Diode_SMD:D_SMA
- IC1: footprint SOIC127P790X216-8N -> Evan's Kicad Library:SOIC127P790X216-8N
- IC2: footprint SOIC127P600X175-8N -> Evan's Kicad Library:SOIC127P600X175-8N
- J1: footprint CONN_BM03B-SRSS-TBLFSN_JST -> Evan's Kicad Library:CONN_BM03B-SRSS-TBLFSN_JST
- J2, J3: footprint (none) -> Connector_PinHeader_2.54mm:PinHeader_1x20_P2.54mm_Vertical
- J4: footprint (none) -> Evan's Kicad Library:TF-115YY-ACP9
- L1: footprint (none) -> Inductor_SMD:L_1008_2520Metric
- R10, R11, R12, R15, R16, R17, R19, R20, R4, R5, R6, R7, R8, R9: footprint (none) -> Resistor_SMD:R_0603_1608Metric
- TP1, TP10, TP11, TP2, TP3, TP4, TP5, TP6, TP7: footprint (none) -> TestPoint:TestPoint_Pad_1.5x1.5mm
- U1: footprint (none) -> Evan's Kicad Library:RP2350A_QFN-60_EP_7.75x7.75_Pitch0.4mm
- Y1: footprint ECS1202033CKMTR -> Evan's Kicad Library:ECS1202033CKMTR
Connections:
- net GND: no longer SW1.2, SW2.2
- net SW_RESET: now also SW2.2 (K); no longer SW2.3 (K), SW2.4 (A)
- net at R6.1, TP6.1: now also SW1.2 (K); no longer SW1.3 (K), SW1.4 (A)
